File: genesis_s-video_simple.kicad_sch (KiCad schematic)
At the start: 12 parts, among them J1 Y In, J2 C In, J3 +5V, J4 Y Out, J5 C Out, J6 GND, J7 CGND, J8 YGND, Q2 KSC945

Commit message: minor update
slightly shrunk pcb, widened transistor pins for easier installation, and slight silkscreen change
Parts:
- Q2: footprint Package_TO_SOT_THT:TO-92L -> Package_TO_SOT_THT:TO-92L_Inline_Wide
Changed lines of the file:
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@@
       (effects (font (size 1.27 1.27)) (justify left))
     )
-    (property "Footprint" "Package_TO_SOT_THT:TO-92L" (at 62.23 33.02 0)
+    (property "Footprint" "Package_TO_SOT_THT:TO-92L_Inline_Wide" (at 62.23 33.02 0)
       (effects (font (size 1.27 1.27)) hide)
     )
